Commit message: updated launch and xacro

File: urdf/rgb_cam.xacro (robot description, xacro)
@@ -1,4 +1,15 @@
 <?xml version="1.0" ?>
 <robot name="openArm_cam" xmlns:xacro="http://www.ros.org/wiki/xacro">
+	<!-- Use world link for fixing the robot-->
+	<link name="world" />
+	<inertial>
+		<mass value="0.00001" />
+		<origin rpy="0 0 0" xyz="0 0 0" />
+		<inertia ixx="0.0" ixy="0.0" ixz="0.0" iyy="0.0" iyz="0.0" izz="0.0" />
+	</inertial>
+	<joint name="fixed" type="fixed">
+		<parent link="world" />
+		<child link="camera_base" />
+	</joint>
 	<!-- Base Camera Link -->
 	<link name="camera_base">

Commit message: added depth

File: urdf/rgb_cam.xacro (robot description, xacro)
@@ -8,64 +8,72 @@
 		<inertia ixx="0.0" ixy="0.0" ixz="0.0" iyy="0.0" iyz="0.0" izz="0.0" />
 	</inertial>
-	<joint name="fixed" type="fixed">
-		<parent link="world" />
-		<child link="camera_base" />
-	</joint>
-	<!-- Base Camera Link -->
-	<link name="camera_base">
-	<inertial>
-		<origin xyz="0 0 0" rpy="0 0 0" />
-		<mass value="0.001" />
-		<inertia ixx="0.000001" ixy="0.0" ixz="0.0" iyy="0.000001" iyz="0.0" izz="0.000001" />
-	</inertial>
-	<visual>
-		<origin rpy="0.0 0 0" xyz="0 0 0" />
-		<geometry>
-			<box size="0.0005 0.0005 0.0005" />
-		</geometry>
-	</visual>
-	</link>
-	<!-- Camera Sensor -->
-	<sensor name="arm_cam" update_rate="20">
-		<parent link="camera_base" />
-		<origin xyz="0 0 0" rpy="0 0 0" />
-		<camera>
-			<image width="1920" height="1080" hfov="1.467822" format="RGB8" near="0.05" far="10" />
-		</camera>
-	</sensor>
-	<!-- Camera Gazebo -->
-	<gazebo reference="camera_base">
-		<sensor type="camera" name="camera1">
-			<always_on>true</always_on>
-			<visualize>true</visualize>
-			<update_rate>15.0</update_rate>
-			<camera name="arm_cam">
-				<pose>0 0 0 0 0 1.57</pose>
-				<horizontal_fov>1.467822</horizontal_fov>
-				<image>
-					<width>1920</width>
-					<height>1080</height>
-					<format>R8G8B8</format>
-				</image>
-				<clip>
-					<near>0.05</near>
-					<far>10</far>
-				</clip>
-			</camera>
-			<plugin name="camera_controller" filename="libgazebo_ros_camera.so">
-				<alwaysOn>true</alwaysOn>
-				<updateRate>0.0</updateRate>
-				<cameraName>openArm_cam/camera1</cameraName>
-				<imageTopicName>image_raw</imageTopicName>
-				<cameraInfoTopicName>camera_info</cameraInfoTopicName>
-				<frameName>camera_link</frameName>
-				<hackBaseline>0.0</hackBaseline>
-				<distortionK1>0.0</distortionK1>
-				<distortionK2>0.0</distortionK2>
-				<distortionK3>0.0</distortionK3>
-				<distortionT1>0.0</distortionT1>
-				<distortionT2>0.0</distortionT2>
-			</plugin>
-		</sensor>
-	</gazebo>
+<link name="camera">
+    <collision>
+      <origin xyz="0 0 0" rpy="0 0 0"/>
+      <geometry>
+        <box size="0.1 0.3 0.3"/>
+      </geometry>
+    </collision>
+    <visual>
+      <origin xyz="0 0 0" rpy="0 0 0"/>
+      <geometry>
+        <box size="0.1 0.3 0.3 "/>
+      </geometry>
+    </visual>
+    <inertial>
+      <mass value="1" />
+      <origin xyz="0 0 0" rpy="0 0 0"/>
+      <inertia ixx="1e-6" ixy="0" ixz="0" iyy="1e-6" iyz="0" izz="1e-6" />
+    </inertial>
+  </link>
+  <joint name="camera_joint" type="fixed">
+    <axis xyz="0 1 0" />
+    <origin xyz="0 0 0" rpy="0 0 0"/>
+    <parent link="world"/>
+    <child link="camera"/>
+  </joint>
+<gazebo reference="camera">
+  <static>true</static>
+</gazebo>
+<gazebo reference="camera">
+  <sensor name="depth_camera" type="depth">
+    <update_rate>20</update_rate>
+    <camera>
+      <horizontal_fov>1.047198</horizontal_fov>
+      <image>
+        <width>640</width>
+        <height>480</height>
+        <format>R8G8B8</format>
+      </image>
+      <clip>
+        <near>0.05</near>
+        <far>3</far>
+      </clip>
+    </camera>
+    <plugin name="camera_controller" filename="libgazebo_ros_openni_kinect.so">
+      <baseline>0.2</baseline>
+      <alwaysOn>true</alwaysOn>
+      <updateRate>1.0</updateRate>
+      <cameraName>depth_camera_ir</cameraName>
+      <imageTopicName>depth_camera/color/image_raw</imageTopicName>
+      <cameraInfoTopicName>depth_camera/color/camera_info</cameraInfoTopicName>
+      <depthImageTopicName>depth_camera/depth/image_raw</depthImageTopicName>
+      <depthImageInfoTopicName>depth_camera/depth/camera_info</depthImageInfoTopicName>
+      <pointCloudTopicName>depth_camera/depth/points</pointCloudTopicName>
+      <frameName>depth_frame</frameName>
+      <pointCloudCutoff>0.2</pointCloudCutoff>
+      <pointCloudCutoffMax>3.0</pointCloudCutoffMax>
+      <distortionK1>0.00000001</distortionK1>
+      <distortionK2>0.00000001</distortionK2>
+      <distortionK3>0.00000001</distortionK3>
+      <distortionT1>0.00000001</distortionT1>
+      <distortionT2>0.00000001</distortionT2>
+      <CxPrime>0</CxPrime>
+      <Cx>0</Cx>
+      <Cy>0</Cy>
+      <focalLength>0</focalLength>
+      <hackBaseline>0</hackBaseline>
+    </plugin>
+  </sensor>
+</gazebo>
 </robot>
